Commit message: Add robot_localization to bringup_only_navigation.launch

File: kobuki_gazebo_melodic/src/itri_multi_robot_kobuki/itri_robot_description/urdf/kobuki/gazebo/itri_gpu_hokuyo_gazebo.urdf.xacro (robot description, xacro)
@@ -4,16 +4,16 @@
   <!--xacro:include filename="/home/lui/Documents/multi_turtlebot_2/turtlebot _gazebo.urdf.xacro"/-->
   <xacro:include filename="$(find turtlebot_description)/urdf/turtlebot_properties.urdf.xacro"/>
-  <xacro:include filename="$(find itri_robot_gazebo)/urdf/hokuyo_gazebo.urdf.xacro"/>
+  <xacro:include filename="$(find itri_robot_gazebo)/urdf/gpu_hokuyo_gazebo.urdf.xacro"/>
   <!-- 2D LIDAR -->
-  <xacro:macro name="sensor_hokuyo" params="parent">
-    <joint name="laser" type="fixed">
+  <xacro:macro name="sensor_gpu_hokuyo" params="parent">
+    <joint name="gpu_laser" type="fixed">
       <!-- <origin xyz="0.0 0.0 0.035" rpy="0 0.0 0.0" /> -->
       <!-- <parent link="plate_top_link" /> -->
       <origin xyz="0.0 0 0.435" rpy="0 0.0 0.0" />
       <parent link="base_link"/>
-      <child link="hokuyo_link" />
+      <child link="hokuyo_gpu_link" />
     </joint>
-    <!-- Hokuyo Laser -->
-    <link name="hokuyo_link">
+    <!-- Hokuyo GPU Laser -->
+    <link name="hokuyo_gpu_link">
       <collision>
         <origin xyz="0 0 0" rpy="0 0 0"/>
@@ -33,8 +33,8 @@
         <origin xyz="0 0 0" rpy="0 0 0"/>
         <inertia ixx="1e-6" ixy="0" ixz="0" iyy="1e-6" iyz="0" izz="1e-6" />
-        </inertial>
+      </inertial>
     </link>
     <!-- Set up laser gazebo details -->
-    <turtlebot_sim_2d_laser/>
+    <turtlebot_sim_2d_gpu_laser/>
   </xacro:macro>
 </robot>

File: kobuki_gazebo_melodic/src/itri_multi_robot_kobuki/itri_robot_description/urdf/kobuki/gazebo/itri_robot_gazebo.urdf.xacro (robot description, xacro)
@@ -10,6 +10,8 @@
   <xacro:include filename="$(find itri_robot_description)/urdf/kobuki/itri_kobuki_base.urdf.xacro" />
   <xacro:include filename="$(find itri_robot_description)/urdf/kobuki/gazebo/itri_hokuyo_gazebo.urdf.xacro"/>
+  <xacro:include filename="$(find itri_robot_description)/urdf/kobuki/gazebo/itri_gpu_hokuyo_gazebo.urdf.xacro"/>
   <kobuki/>
   <stack_hexagons                 parent="base_link"/>
-  <sensor_hokuyo          	      parent="base_link"/>
+  <sensor_gpu_hokuyo          	      parent="base_link"/>
+  <!-- <sensor_hokuyo          	      parent="base_link"/> -->
 </robot>

File: kobuki_gazebo_melodic/src/itri_multi_robot_kobuki/itri_robot_description/urdf/kobuki/itri_robot.urdf.xacro (robot description, xacro)
@@ -10,6 +10,8 @@
   <xacro:include filename="$(find itri_robot_description)/urdf/kobuki/itri_kobuki_base.urdf.xacro" />
   <xacro:include filename="$(find itri_robot_description)/urdf/kobuki/itri_hokuyo.urdf.xacro"/>
+  <xacro:include filename="$(find itri_robot_description)/urdf/kobuki/itri_gpu_hokuyo.urdf.xacro"/>
   <kobuki/>
   <stack_hexagons                 parent="base_link"/>
-  <sensor_hokuyo          	      parent="base_link"/>
+  <!-- <sensor_hokuyo          	      parent="base_link"/> -->
+  <sensor_gpu_hokuyo          	      parent="base_link"/>
 </robot>

File: kobuki_gazebo_melodic/src/itri_multi_robot_kobuki/itri_robot_gazebo/urdf/gpu_hokuyo_gazebo.urdf.xacro (robot description, xacro)
@@ -1,9 +1,9 @@
 <?xml version="1.0"?>
 <robot name="hokuyo_gazebo" xmlns:xacro="http://ros.org/wiki/xacro">
-  <xacro:macro name="turtlebot_sim_2d_laser">
-    <gazebo reference="hokuyo_link">
-      <sensor type="ray" name="head_hokuyo_sensor">
+  <xacro:macro name="turtlebot_sim_2d_gpu_laser">
+    <gazebo reference="hokuyo_gpu_link">
+      <sensor type="gpu_ray" name="head_hokuyo_sensor">
         <pose>0 0 0 0 0 0</pose>
-        <visualize>false</visualize>
+        <visualize>true</visualize>
         <update_rate>40</update_rate>
         <ray>
@@ -23,12 +23,12 @@
           <noise>
             <type>gaussian</type>
-              <mean>0.0</mean>
+            <mean>0.0</mean>
             <stddev>0.01</stddev>
           </noise>
         </ray>
-          <plugin name="gazebo_ros_hokuyo_controller" filename="libgazebo_ros_laser.so">
-          <topicName>scan</topicName>
-          <frameName>hokuyo_link</frameName>
-      </plugin>
+        <plugin name="gazebo_ros_gpu_hokuyo_controller" filename="libgazebo_ros_gpu_laser.so">
+          <topicName>gpu_scan</topicName>
+          <frameName>hokuyo_gpu_link</frameName>
+        </plugin>
       </sensor>
     </gazebo>
